File: PCB/RadarProject.kicad_pcb (KiCad board)
At the start: 4 copper layers, 85 x 49 mm, 65 parts, among them J1 Conn_Coaxial, J2 Conn_Coaxial, J3 Conn_01x05, Q1 2N7000, SW1 SW_SPDT, U1 AT0603T03ECATD, U2 PD2328J5050S2HF, U3 BGU8052, U4 BGU8052, U5 RQRA-2328-2536-CR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

Commit message: Final schematic is generally done, just some minor fixes
Parts:
- added R31: 100k, Resistor_SMD:R_0805_2012Metric, F.Cu at (72.0, 30.5)
- added R32: 10k, Resistor_SMD:R_0805_2012Metric, F.Cu at (51.5, 43.2)
- added R33: 10k, Resistor_SMD:R_0805_2012Metric, F.Cu at (55.2, 43.2)
- C11: value 10 nF -> 8 nF
- Q1: value 2N7000 -> Q_NPN_BCE; footprint Package_TO_SOT_THT:TO-92_Inline -> Package_TO_SOT_THT:TO-92L_Inline
- R10, R11, R9: value 49.9k -> 51.1k
- R15: value 100k -> 1k
- R16: value 100k -> 200k
- R18: value 700k -> 100k
- R19: value 500k -> 100k
- moved R29 17.6 mm to (58.8, 46.7)
- moved R9 16.8 mm to (62.6, 32.5), turned to -90 degrees
- moved R16 15.2 mm to (46.9, 41.8), turned to 90 degrees
- moved Q1 14.8 mm to (46.9, 45.4), turned to -90 degrees
- moved R8 13.9 mm to (57.2, 30.9)
- moved C11 13.7 mm to (59.0, 33.2)
- moved R30 12.5 mm to (58.8, 43.2)
- moved R15 10.5 mm to (52.6, 33.1), turned to 180 degrees
- moved RV1 10.1 mm to (56.8, 25.8)
- moved R11 9.92 mm to (63.5, 35.9), turned to 180 degrees
- moved R18 9.27 mm to (48.8, 31.0), turned to 0 degrees
- moved R10 9.05 mm to (55.2, 46.7), turned to 0 degrees
- moved R19 5.32 mm to (52.6, 31.0), turned to 0 degrees
- moved U7 3.50 mm to (55.5, 38.3), turned to -90 degrees
- moved J1 2.50 mm to (102.0, 32.5)
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Connections:
- Q1 pad 1: Earth -> Net-(Q1-Pad1)
- Q1 pad 3: Net-(Q1-Pad3) -> Earth
- R10 pad 1: Net-(Q1-Pad3) -> Net-(Q1-Pad2)
- R15 pad 2: Net-(Q1-Pad2) -> Net-(R15-Pad2)
- R16 pad 1: Net-(C11-Pad2) -> Net-(Q1-Pad1)
- R16 pad 2: Net-(R16-Pad2) -> Net-(R15-Pad2)
- R18 pad 1: Net-(R16-Pad2) -> +5V
- R18 pad 2: Earth -> Net-(R15-Pad1)
- R19 pad 1: Net-(R16-Pad2) -> Earth
- R19 pad 2: +5V -> Net-(R15-Pad1)
- SW1 pad 1: Earth -> Net-(R31-Pad2)
- SW1 pad 2: Net-(SW1-Pad2) -> Net-(C11-Pad2)
- U7 pad 10: Net-(R16-Pad2) -> Net-(R32-Pad2)
- U7 pad 7: Net-(Q1-Pad2) -> Net-(R15-Pad2)
- U7 pad 8: Net-(SW1-Pad2) -> Net-(U7-Pad8)
- U7 pad 9: Net-(SW1-Pad2) -> Net-(U7-Pad8)
Routing:
- net Net-(C11-Pad1): track 46.0 -> 20.6 mm, vias 0 -> 2
- net Net-(SW1-Pad2): track 17.5 -> 0.00 mm
- net Net-(C11-Pad2): track 39.8 -> 25.8 mm
- net Net-(R16-Pad2): track 13.7 -> 0.00 mm
- net Net-(R15-Pad2): track 0.00 -> 11.0 mm
- net Net-(R29-Pad2): track 15.8 -> 6.34 mm
- net Net-(Q1-Pad3): track 5.44 -> 0.00 mm
- net Net-(R8-Pad1): track 9.13 -> 13.8 mm
- net Net-(R32-Pad2): track 0.00 -> 4.25 mm
- net Net-(R31-Pad2): track 0.00 -> 3.84 mm
- net +5V: track 53.6 -> 56.5 mm, vias 13 -> 14
- net Net-(Q1-Pad1): track 0.00 -> 2.68 mm
- net Earth: track 104.1 -> 106.7 mm, vias 17 -> 15
- net Net-(C4-Pad1): track 12.5 -> 15.1 mm
- net Net-(J2-Pad1): track 67.3 -> 69.8 mm
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- removed copper zone on In2.Cu, net Earth

Commit message: Updated PCB, added antennas, etc.
Parts:
- moved R31 11.0 mm to (62.0, 25.9), turned to -90 degrees
- moved U1 3.05 mm to (34.8, 41.7)
- moved U5 3.05 mm to (27.7, 24.6)
Connections:
- R31 pad 1: Earth -> Net-(R31-Pad1)
- R31 pad 2: Net-(R31-Pad2) -> Earth
- SW1 pad 1: Net-(R31-Pad2) -> Net-(C11-Pad2)
- SW1 pad 2: Net-(C11-Pad2) -> Net-(J3-Pad5)
- SW1 pad 3: Net-(J3-Pad5) -> Net-(R31-Pad1)
Routing:
- net Earth: track 106.7 -> 129.9 mm, vias 15 -> 18
- net Net-(R31-Pad1): track 0.00 -> 9.62 mm
- net Net-(C11-Pad1): track 20.6 -> 25.5 mm
- net Net-(R31-Pad2): track 3.84 -> 0.00 mm
- net Net-(C2-Pad1): track 9.69 -> 12.7 mm
- net Net-(J3-Pad5): track 83.5 -> 80.5 mm
- net Net-(C11-Pad2): track 25.8 -> 28.2 mm
- net Net-(C12-Pad1): track 18.1 -> 19.9 mm
- net Net-(R3-Pad1): track 7.61 -> 8.65 mm
- net Net-(J2-Pad1): track 69.8 -> 70.7 mm
- net Net-(C14-Pad1): track 19.5 -> 20.1 mm
- added copper zone on In1.Cu, net +5V
- added copper zone on In2.Cu, net Earth
Other:
- board text added: "RX"
- board text added: "TX"

Commit message: Final production PCB
Routing:
- net Earth: track 129.9 -> 128.3 mm, vias 18 -> 17
- removed copper zone on In1.Cu, net +5V
- removed copper zone on In2.Cu, net Earth
Other:
- board text added: "Behold, my latest fire hazard!"
- board text added: "CRISPR ME SOME CAT EARS!"
- board text added: "Dan Seal of Approval"
- board text added: "God likes elephants, and I like elephants"
- board text added: "Order copies JLC PCB 4 Layers JLC7628"
- board text added: "This is unhealthy."
Changed lines of the file:
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@@
     (property "Sheetname" "")
     (attr smd)
-    (fp_text reference "R6" (at 0 -1.65 90) (layer "F.SilkS")
+    (fp_text reference "R6" (at 0.9325 -1.99 180) (layer "F.SilkS")
       (effects (font (size 1 1) (thickness 0.15)))
     )
@@
     (property "Sheetname" "")
     (attr through_hole)
-    (fp_text reference "RV1" (at -2.54 -3.66) (layer "F.SilkS")
+    (fp_text reference "RV1" (at -9.25 -0.0775) (layer "F.SilkS")
       (effects (font (size 1 1) (thickness 0.15)))
     )
@@
     (property "Sheetname" "")
     (attr through_hole)
-    (fp_text reference "J3" (at -0.01 13.5 180) (layer "F.SilkS")
+    (fp_text reference "J3" (at 1.37 -2.83 180) (layer "F.SilkS")
       (effects (font (size 1 1) (thickness 0.15)))
     )
@@
     (property "Sheetname" "")
     (attr exclude_from_pos_files)
-    (fp_text reference "H2" (at -3.68 2.03) (layer "F.SilkS")
+    (fp_text reference "H2" (at -3.32 -2.67) (layer "F.SilkS")
       (effects (font (size 1 1) (thickness 0.15)))
     )
@@
     (property "Sheetname" "")
     (attr smd)
-    (fp_text reference "U5" (at 3.73 -2.37 unlocked) (layer "F.SilkS")
+    (fp_text reference "U5" (at -1.1 1.09 unlocked) (layer "F.SilkS")
       (effects (font (size 1 1) (thickness 0.15)))
     )
@@
   (gr_line (start 20 23) (end 20 66) (layer "Edge.Cuts") (width 0.1))
   (gr_arc (start 20 23) (mid 20.87868 20.87868) (end 23 20) (layer "Edge.Cuts") (width 0.1))
-  (gr_text "Sckzor's 2.4GHz Radar" (at 53.88 53.07) (layer "F.SilkS")
+  (gr_text "CRISPR ME \nSOME\nCAT EARS!" (at 34.45 31.31) (layer "F.SilkS")
+    (effects (font (size 1 1) (thickness 0.15)))
+  )
+  (gr_text "Sckzor's 2.4GHz Radar" (at 53.82 53.78) (layer "F.SilkS")
+    (effects (font (size 1.778 1.778) (thickness 0.381)))
+  )
+  (gr_text "This is unhealthy." (at 91.92 66.48) (layer "F.SilkS")
+    (effects (font (size 1 1) (thickness 0.15)))
+  )
+  (gr_text "Behold, my latest fire hazard!" (at 44.26 21.86) (layer "F.SilkS")
     (effects (font (size 1.5 1.5) (thickness 0.3)))
+  )
+  (gr_text "God likes\nelephants,\nand I like \nelephants\n" (at 26.69 42.91) (layer "F.SilkS")
+    (effects (font (size 1 1) (thickness 0.15)))
   )
   (gr_text "TX" (at 101.94 49.44) (layer "F.SilkS")
@@
   (gr_text "RX" (at 101.94 39.7) (layer "F.SilkS")
     (effects (font (size 2 2) (thickness 0.15)))
+  )
+  (gr_text "Dan Seal of\nApproval" (at 45 57.79) (layer "F.SilkS")
+    (effects (font (size 1.016 1.016) (thickness 0.1778)))
+  )
+  (gr_text "Order copies\nJLC PCB\n4 Layers\nJLC7628" (at 72.22 34.39) (layer "F.SilkS")
+    (effects (font (size 1 1) (thickness 0.15)))
   )
   (segment (start 78.51 28.92) (end 80.08 28.92) (width 0.293) (layer "F.Cu") (net 1))
@@
   (segment (start 27.7 27.56) (end 30.61 24.65) (width 0.293) (layer "F.Cu") (net 1))
   (segment (start 32.27 37.35) (end 29.73 37.35) (width 0.293) (layer "F.Cu") (net 1))
-  (segment (start 64.56 55.97) (end 64.56 58.31) (width 0.25) (layer "F.Cu") (net 1))
   (segment (start 89.61 26.94) (end 91.215 26.94) (width 0.293) (layer "F.Cu") (net 1))
+  (segment (start 36.505 42.745) (end 37.35 41.9) (width 0.25) (layer "F.Cu") (net 1))
   (segment (start 46.6825 66.96625) (end 46.5975 66.88125) (width 0.25) (layer "F.Cu") (net 1))
   (segment (start 55.55 38.68) (end 55.55 40.795) (width 0.293) (layer "F.Cu") (net 1))
@@
   (segment (start 102 43.68) (end 102 52.25) (width 0.293) (layer "F.Cu") (net 1))
   (segment (start 46.0225 66.6125) (end 46.0225 66.39125) (width 0.25) (layer "F.Cu") (net 1))
+  (segment (start 37.35 41.9) (end 37.35 37.35) (width 0.25) (layer "F.Cu") (net 1))
   (segment (start 35.69 24.65) (end 38.23 24.65) (width 0.293) (layer "F.Cu") (net 1))
   (segment (start 55.5325 40.8125) (end 55.5325 42.635) (width 0.293) (layer "F.Cu") (net 1))
+  (segment (start 34.82 42.745) (end 36.505 42.745) (width 0.25) (layer "F.Cu") (net 1))
   (segment (start 36.6375 63.565) (end 38.785 63.565) (width 0.293) (layer "F.Cu") (net 1))
   (segment (start 40.4 32.4) (end 40.4 34.94) (width 0.293) (layer "F.Cu") (net 1))
@@
   (segment (start 38.785 63.565) (end 40.8625 63.565) (width 0.293) (layer "F.Cu") (net 1))
   (segment (start 25.58625 62.43625) (end 25.59 62.44) (width 0.25) (layer "F.Cu") (net 1))
-  (segment (start 34.82 42.745) (end 35.275 42.745) (width 0.25) (layer "F.Cu") (net 1))
   (segment (start 29.44625 52.555) (end 29.19625 52.805) (width 0.25) (layer "F.Cu") (net 1))
   (segment (start 55.55 40.795) (end 55.5325 40.8125) (width 0.25) (layer "F.Cu") (net 1))
@@
   (segment (start 38.785 62.265) (end 38.785 63.565) (width 0.293) (layer "F.Cu") (net 1))
   (segment (start 40.4 24.65) (end 40.4 27.32) (width 0.293) (layer "F.Cu") (net 1))
-  (segment (start 35.275 42.745) (end 37.35 40.67) (width 0.25) (layer "F.Cu") (net 1))
-  (segment (start 37.35 40.67) (end 37.35 37.35) (width 0.25) (layer "F.Cu") (net 1))
   (segment (start 45.3625 67.38125) (end 45.3625 66.96625) (width 0.25) (layer "F.Cu") (net 1))
   (segment (start 30.19625 52.555) (end 29.44625 52.555) (width 0.293) (layer "F.Cu") (net 1))
@@
   (via (at 61.97 28.42) (size 0.8) (drill 0.4) (layers "F.Cu" "B.Cu") (net 1))
   (via (at 25.61 62.28) (size 0.8) (drill 0.4) (layers "F.Cu" "B.Cu") (net 1))
-  (via (at 78.51 28.92) (size 0.8) (drill 0.4) (layers "F.Cu" "B.Cu") (net 1))
+  (via (at 78.51 28.92) (size 0.8) (drill 0.4) (layers "F.Cu" "B.Cu") (remove_unused_layers) (keep_end_layers) (net 1))
   (via (at 76.54 46.22) (size 0.8) (drill 0.4) (layers "F.Cu" "B.Cu") (net 1))
   (via (at 40.86 64.92) (size 0.8) (drill 0.4) (layers "F.Cu" "B.Cu") (net 1))
@@
   (via (at 98.14 60.75) (size 0.8) (drill 0.4) (layers "F.Cu" "B.Cu") (free) (net 1))
   (via (at 91.24 26.94) (size 0.8) (drill 0.4) (layers "F.Cu" "B.Cu") (net 1))
-  (via (at 64.56 55.97) (size 0.8) (drill 0.4) (layers "F.Cu" "B.Cu") (net 1))
   (via (at 27.7 37.35) (size 0.8) (drill 0.4) (layers "F.Cu" "B.Cu") (remove_unused_layers) (keep_end_layers) (net 1))
   (segment (start 92.1775 49.5) (end 92.17 49.5075) (width 0.25) (layer "F.Cu") (net 2))
@@
   (via (at 50.57 45.17) (size 0.8) (drill 0.4) (layers "F.Cu" "B.Cu") (remove_unused_layers) (keep_end_layers) (free) (net 2))
   (via (at 85.62 60.97) (size 0.8) (drill 0.4) (layers "F.Cu" "B.Cu") (free) (net 2))
-  (via (at 81.24 34.14) (size 0.8) (drill 0.4) (layers "F.Cu" "B.Cu") (free) (net 2))
+  (via (at 81.24 34.14) (size 0.8) (drill 0.4) (layers "F.Cu" "B.Cu") (remove_unused_layers) (keep_end_layers) (free) (net 2))
   (via (at 95.19 49.5) (size 0.8) (drill 0.4) (layers "F.Cu" "B.Cu") (free) (net 2))
   (via (at 61.36 46.69) (size 0.8) (drill 0.4) (layers "F.Cu" "B.Cu") (free) (net 2))
@@
   (segment (start 51.7225 40.8125) (end 52.9925 40.8125) (width 0.293) (layer "F.Cu") (net 57))
   (segment (start 58.0725 40.8125) (end 59.3425 40.8125) (width 0.293) (layer "F.Cu") (net 58))
-  (zone (net 2) (net_name "+5V") (layers "In1.Cu" "In2.Cu") (name "5v") (hatch edge 0.508)
+  (zone (net 1) (net_name "Earth") (layer "In1.Cu") (hatch full 0.508)
     (connect_pads (clearance 0.508))
     (min_thickness 0.254) (filled_areas_thickness no)
@@
     (polygon
       (pts
+        (xy 105 68.99)
+        (xy 20 69)
+        (xy 20 20)
         (xy 105 20)
-        (xy 105 69)
-        (xy 20 69)
-        (xy 20.01 19.99)
       )
     )
   )
-  (zone (net 1) (net_name "Earth") (layers "In1.Cu" "In2.Cu") (hatch edge 0.508)
+  (zone (net 2) (net_name "+5V") (layer "In2.Cu") (hatch edge 0.508)
     (connect_pads (clearance 0.508))
     (min_thickness 0.254) (filled_areas_thickness no)

Commit message: new version of PCB
Parts:
- removed R29, R30: 10k, Resistor_SMD:R_0805_2012Metric
- added REF**: OSHW-Logo2_9.8x8mm_SilkScreen, Symbol:OSHW-Logo2_9.8x8mm_SilkScreen, F.Cu at (69.0, 42.8)
- J1, J2: footprint Connector_Coaxial:SMA_Amphenol_132289_EdgeMount -> Connector_Coaxial:SMA_Samtec_SMA-J-P-X-ST-EM1_EdgeMount
- U5: value RQRA-2328-2536-CR -> CVCO55CC-2230-2430; footprint RadarProject:RQRA-2328-2536-CR -> RadarProject:CVCO55CC-2230-2430
- moved U5 18.8 mm to (40.5, 38.4), turned to 180 degrees
- moved C8 13.1 mm to (79.7, 30.4), turned to 180 degrees
- moved C4 10.7 mm to (81.8, 22.9), turned to -90 degrees
- moved C6 10.5 mm to (91.4, 30.4), turned to 180 degrees
- moved C1 8.36 mm to (33.3, 56.8)
- moved C3 7.91 mm to (89.8, 25.7), turned to 180 degrees
- moved R1 7.85 mm to (33.3, 52.9)
- moved C7 7.57 mm to (30.4, 56.6), turned to -90 degrees
- moved L1 7.54 mm to (26.7, 56.7)
- moved U4 6.05 mm to (82.6, 25.7), turned to -90 degrees
- moved R4 5.21 mm to (25.7, 59.8)
- moved C5 4.70 mm to (26.7, 62.7)
- moved C2 4.31 mm to (30.4, 47.9)
- moved L2 4.31 mm to (84.1, 30.4), turned to 180 degrees
- moved U3 3.49 mm to (31.2, 52.0), turned to -90 degrees
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Connections:
- Q1 pad 1: Net-(Q1-Pad1) -> Earth
- Q1 pad 2: Net-(Q1-Pad2) -> Net-(R16-Pad1)
- Q1 pad 3: Earth -> Net-(R10-Pad1)
- R10 pad 1: Net-(Q1-Pad2) -> Net-(R10-Pad1)
- R16 pad 1: Net-(Q1-Pad1) -> Net-(R16-Pad1)
- SW1 pad 1: Net-(C11-Pad2) -> Net-(U7-Pad13)
- U7 pad 12: Net-(R29-Pad2) -> Net-(C11-Pad2)
Routing:
- net Earth: track 128.3 -> 104.0 mm
- net Net-(U7-Pad13): track 1.27 -> 23.6 mm
- net Net-(AE2-Pad2): track 0.00 -> 21.8 mm
- net Net-(C8-Pad2): track 81.3 -> 68.0 mm
- net Net-(C4-Pad1): track 15.1 -> 28.3 mm
- net Net-(C11-Pad2): track 28.2 -> 15.6 mm, vias 2 -> 0
- net Net-(C2-Pad1): track 12.7 -> 4.35 mm
- net Net-(R16-Pad1): track 0.00 -> 8.03 mm
- net Net-(R10-Pad1): track 0.00 -> 7.91 mm
- net Net-(Q1-Pad2): track 7.38 -> 0.00 mm
- net Net-(C7-Pad2): track 31.6 -> 24.9 mm
- net Net-(R29-Pad2): track 6.34 -> 0.00 mm
- net +5V: track 56.5 -> 51.7 mm, vias 14 -> 12
- net Net-(AE1-Pad2): track 0.00 -> 3.81 mm
- net Net-(C5-Pad2): track 7.22 -> 3.92 mm
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Other:
- board text added: "Barfunkel Endorced"
- board text added: "JLCJLCJLCJLC"
- board text added: "Revision Mk. II"
- board text added: "on the line at: www.sckz.org"
