File: AnalogRadar/MkII/RadarProject.kicad_pcb (KiCad board)
At the start: 4 copper layers, 85 x 49 mm, 67 parts, among them J1 Conn_Coaxial, J2 Conn_Coaxial, J3 Conn_01x05, Q1 Q_NPN_BCE, SW1 SW_SPDT, U1 AT0603T03ECATD, U2 PD2328J5050S2HF, U3 BGU8052, U4 BGU8052, U5 CVCO55CC-2230-2430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

Commit message: Updated PCB designs
Parts:
- removed R27: 10k, Resistor_SMD:R_0805_2012Metric
- removed R28: 50, Resistor_SMD:R_0805_2012Metric
- moved J2 83.4 mm to (102.0, 56.5), turned to 90 degrees
- moved J1 83.4 mm to (102.0, 32.5), turned to 90 degrees
- moved C3 67.5 mm to (89.8, 25.7), turned to 180 degrees
- moved R2 64.7 mm to (85.5, 25.7), turned to 180 degrees
- moved C4 64.6 mm to (81.8, 22.9), turned to -90 degrees
- moved U4 62.6 mm to (82.6, 25.7), turned to -90 degrees
- moved C6 61.3 mm to (91.4, 30.4)
- moved R5 60.2 mm to (87.7, 29.5)
- moved R13 59.1 mm to (95.2, 45.8), turned to -90 degrees
- moved L2 57.7 mm to (84.1, 30.4), turned to 180 degrees
- moved C12 56.7 mm to (91.2, 49.5), turned to 0 degrees
- moved C8 55.5 mm to (79.7, 30.4), turned to 180 degrees
- moved R14 53.7 mm to (90.3, 45.8), turned to -90 degrees
- moved R7 53.2 mm to (87.5, 59.2), turned to 90 degrees
- moved C9 52.4 mm to (88.4, 54.8), turned to 180 degrees
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Connections:
- C9 pad 2: Net-(R7-Pad1) -> Net-(C9-Pad2)
- J2 pad 2: Earth -> Net-(AE2-Pad2)
- R7 pad 1: Net-(R7-Pad1) -> +5V
- R7 pad 2: Earth -> Net-(C9-Pad2)
- U6 pad 5: Net-(U6-Pad5) -> Net-(C9-Pad1)
- U8 pad 10: Net-(R7-Pad1) -> Net-(C9-Pad2)
Routing:
- net Earth: track 11.5 -> 104.0 mm, vias 615 -> 16
- net Net-(C9-Pad1): track 1.86 -> 67.2 mm
- net Net-(J2-Pad1): track 7.36 -> 70.7 mm
- net Net-(C8-Pad2): track 7.96 -> 68.0 mm
- net Net-(J3-Pad5): track 36.8 -> 79.2 mm
- net +5V: track 22.5 -> 48.1 mm, vias 17 -> 11
- net Net-(C4-Pad1): track 3.83 -> 28.3 mm
- net Net-(C10-Pad2): track 36.6 -> 13.4 mm
- net Net-(C7-Pad2): track 2.20 -> 25.2 mm
- net Net-(AE1-Pad2): track 0.00 -> 22.2 mm
- net Net-(R7-Pad1): track 17.4 -> 0.00 mm
- net Net-(R17-Pad2): track 25.0 -> 8.61 mm
- net Net-(R26-Pad2): track 7.66 -> 23.6 mm
- net Net-(C14-Pad1): track 4.70 -> 20.1 mm, vias 0 -> 2
- net Net-(SW1-Pad1): track 9.47 -> 23.6 mm
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- removed copper zone on F.Cu, net Earth
Other:
- board text added: "Revision Mk. II"
- board text removed: "Revision Mk. III"
