File: AnalogRadar/MkII/RadarProject.kicad_sch (KiCad schematic)
At the start: 68 parts, among them J1 Conn_Coaxial, J2 Conn_Coaxial, J3 Conn_01x05, Q1 Q_NPN_BCE, SW1 SW_SPDT, U1 AT0603T03ECATD, U2 PD2328J5050S2HF, U3 BGU8052, U4 BGU8052, U5 CVCO55CC-2230-2430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

Commit message: Updated PCB designs
Parts:
- removed R27: 10k, Resistor_SMD:R_0805_2012Metric, symbol Device:R
- removed R28: 50, Resistor_SMD:R_0805_2012Metric, symbol Device:R
Connections:
- net +5V: now also R7.1
- net Earth: no longer R7.2
- net at C9.2, U8.10 (+): now also R7.2; no longer R7.1
- net at C9.1: now also U6.5 (IF)
Other:
- moved on the sheet: R7, U8E
